File: hardware/drone/audio.kicad_sch (KiCad schematic)
At the start: 20 parts, among them U11 TAC5111IRGER, U12 LM4670SD/NOPB

Commit message: More footprints
Parts:
- removed LS1: Speaker, symbol Device:Speaker
- removed U12: LM4670SD/NOPB, Package_SON:WSON-8-1EP_3x3mm_P0.5mm_EP1.6x2.0mm, symbol SoftDrone:LM4670SD/NOPB
- added C97: 100n, Capacitor_SMD:C_0603_1608Metric, symbol Device:C
- added J6: Conn_01x02_Socket, Connector_JST:JST_SH_BM02B-SRSS-TB_1x02-1MP_P1.00mm_Vertical, symbol Connector:Conn_01x02_Socket
- added U28: LM4670ITL/NOPB, LM4670ITL_NOPB:BGA9C50P3X3_146X148X68, symbol SoftDrone:LM4670ITL/NOPB
- C66, C70, C71, C75: footprint (none) -> Capacitor_SMD:C_0402_1005Metric
- C67, C69, C72, C79: footprint (none) -> Capacitor_SMD:C_0805_2012Metric
- C68, C73, C74, C76, C77, C78: footprint (none) -> Capacitor_SMD:C_0603_1608Metric
- R10, R9: footprint (none) -> Resistor_SMD:R_0603_1608Metric
Connections:
- net GND: now also C97.2, U28.A2 (GND), U28.B3 (GND)
- net SPK_EN: now also U28.C2 (~{SHUTDOWN})
- net VSYS_5V: now also C97.1, U28.B1 (VDD), U28.B2 (PVDD)
- net at R9.2: now also U28.C1 (-IN)
- net at R10.2: now also U28.A1 (+IN)
- new net: J6.1 (Pin_1), U28.A3 (VO2)
- new net: J6.2 (Pin_2), U28.C3 (VO1)
Other:
- note added: "20MM-4Ω3W C50387236"
- moved on the sheet: C78, C79

Commit message: Completed footprint assignments
Connections:
- net at J6.1 (Pin_1): now also U28.C3 (VO1); no longer U28.A3 (VO2)
- net at J6.2 (Pin_2): now also U28.A3 (VO2); no longer U28.C3 (VO1)
Changed lines of the file:
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@@
 	(symbol
 		(lib_id "Connector:Conn_01x02_Socket")
-		(at 232.41 80.01 0)
+		(at 232.41 82.55 0)
+		(mirror x)
 		(unit 1)
 		(body_style 1)
@@
 		(in_pos_files yes)
 		(dnp no)
-		(fields_autoplaced yes)
 		(property "Reference" "J6"
-			(at 233.68 80.0099 0)
+			(at 233.68 82.5501 0)
 			(show_name no)
 			(do_not_autoplace no)
@@
 		)
 		(property "Value" "Conn_01x02_Socket"
-			(at 233.68 82.5499 0)
+			(at 233.68 80.0101 0)
 			(show_name no)
 			(do_not_autoplace no)
@@
 		)
 		(property "Footprint" "Connector_JST:JST_SH_BM02B-SRSS-TB_1x02-1MP_P1.00mm_Vertical"
-			(at 232.41 80.01 0)
+			(at 232.41 82.55 0)
 			(hide yes)
 			(show_name no)
@@
 		)
 		(property "Datasheet" ""
-			(at 232.41 80.01 0)
+			(at 232.41 82.55 0)
 			(hide yes)
 			(show_name no)
@@
 		)
 		(property "Description" "Generic connector, single row, 01x02, script generated"
-			(at 232.41 80.01 0)
+			(at 232.41 82.55 0)
 			(hide yes)
 			(show_name no)

Commit message: Labeled nets, added colours, and fixed stm32n6 schematic symbol issues
Connections:
- net CODEC_MEM_IN1P: now reaches C73.2, U11.15 (IN1P)
- net CODEC_MEM_IN1M: now reaches C74.2, U11.16 (IN1M)
- net CODEC_OUT1P: now reaches C76.1, U11.19 (OUT1P)
- net CODEC_OUT1M: now reaches C77.2, U11.20 (OUT1M)
- net CODEC_OUT1P_1: now reaches C76.2, R9.1
- net CODEC_OUT1P_2: now reaches R9.2, U28.C1 (-IN)
- net CODEC_MEM_IN1P_1: now reaches C73.1, MK2.1 (OUT+)
- net CODEC_OUT1M_1: now reaches C77.1, R10.1
- net CODEC_SPK1: now reaches J6.1 (Pin_1), U28.C3 (VO1)
- net CODEC_SPK2: now reaches J6.2 (Pin_2), U28.A3 (VO2)
- net CODEC_OUT1M_2: now reaches R10.2, U28.A1 (+IN)
- net CODEC_MEM_IN1M_1: now reaches C74.1, MK2.3 (OUT-)
Other:
- moved on the sheet: C76, C77
Changed lines of the file:
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@@
 	(wire
 		(pts
-			(xy 180.34 77.47) (xy 180.34 80.01)
+			(xy 181.61 77.47) (xy 181.61 80.01)
 		)
 		(stroke
@@
 	(wire
 		(pts
-			(xy 185.42 82.55) (xy 180.34 82.55)
+			(xy 185.42 82.55) (xy 181.61 82.55)
 		)
 		(stroke
@@
 	(wire
 		(pts
-			(xy 153.67 77.47) (xy 157.48 77.47)
+			(xy 153.67 77.47) (xy 156.21 77.47)
 		)
 		(stroke
@@
 	(wire
 		(pts
-			(xy 165.1 85.09) (xy 168.91 85.09)
-		)
-		(stroke
-			(width 0)
-			(type default)
-		)
-	)
-	(wire
-		(pts
 			(xy 204.47 71.12) (xy 204.47 73.66)
 		)
@@
 	(wire
 		(pts
-			(xy 176.53 77.47) (xy 180.34 77.47)
-		)
-		(stroke
-			(width 0)
-			(type default)
-		)
-	)
-	(wire
-		(pts
-			(xy 180.34 85.09) (xy 176.53 85.09)
+			(xy 176.53 77.47) (xy 181.61 77.47)
+		)
+		(stroke
+			(width 0)
+			(type default)
+		)
+	)
+	(wire
+		(pts
+			(xy 181.61 85.09) (xy 176.53 85.09)
+		)
+		(stroke
+			(width 0)
+			(type default)
+		)
+	)
+	(wire
+		(pts
+			(xy 163.83 85.09) (xy 168.91 85.09)
 		)
 		(stroke
@@
 	(wire
 		(pts
+			(xy 163.83 77.47) (xy 168.91 77.47)
+		)
+		(stroke
+			(width 0)
+			(type default)
+		)
+	)
+	(wire
+		(pts
 			(xy 90.17 62.23) (xy 90.17 60.96)
 		)
@@
 	(wire
 		(pts
-			(xy 180.34 80.01) (xy 185.42 80.01)
+			(xy 181.61 80.01) (xy 185.42 80.01)
 		)
 		(stroke
@@
 	(wire
 		(pts
-			(xy 153.67 85.09) (xy 157.48 85.09)
+			(xy 153.67 85.09) (xy 156.21 85.09)
 		)
 		(stroke
@@
 	(wire
 		(pts
-			(xy 165.1 77.47) (xy 168.91 77.47)
-		)
-		(stroke
-			(width 0)
-			(type default)
-		)
-	)
-	(wire
-		(pts
 			(xy 49.53 58.42) (xy 49.53 74.93)
 		)
@@
 	(wire
 		(pts
+			(xy 207.01 97.79) (xy 204.47 97.79)
+		)
+		(stroke
+			(width 0)
+			(type default)
+		)
+	)
+	(wire
+		(pts
+			(xy 201.93 73.66) (xy 201.93 71.12)
+		)
+		(stroke
+			(width 0)
+			(type default)
+		)
+	)
+	(wire
+		(pts
+			(xy 130.81 52.07) (xy 144.78 52.07)
+		)
+		(stroke
+			(width 0)
+			(type default)
+		)
+	)
+	(wire
+		(pts
 			(xy 59.69 80.01) (xy 69.85 80.01)
 		)
@@
 	(wire
 		(pts
-			(xy 207.01 97.79) (xy 204.47 97.79)
-		)
-		(stroke
-			(width 0)
-			(type default)
-		)
-	)
-	(wire
-		(pts
-			(xy 201.93 73.66) (xy 201.93 71.12)
-		)
-		(stroke
-			(width 0)
-			(type default)
-		)
-	)
-	(wire
-		(pts
-			(xy 130.81 52.07) (xy 144.78 52.07)
-		)
-		(stroke
-			(width 0)
-			(type default)
-		)
-	)
-	(wire
-		(pts
 			(xy 133.35 33.02) (xy 144.78 33.02)
 		)
@@
 	(wire
 		(pts
-			(xy 180.34 82.55) (xy 180.34 85.09)
+			(xy 181.61 82.55) (xy 181.61 85.09)
 		)
 		(stroke
@@
 			(width 0)
 			(type default)
+		)
+	)
+	(label "CODEC_OUT1P_2"
+		(at 176.53 77.47 0)
+		(effects
+			(font
+				(size 0.381 0.381)
+			)
+			(justify left bottom)
+		)
+	)
+	(label "CODEC_OUT1P"
+		(at 148.59 80.01 0)
+		(effects
+			(font
+				(size 0.381 0.381)
+			)
+			(justify left bottom)
+		)
+	)
+	(label "CODEC_OUT1M"
+		(at 148.59 82.55 0)
+		(effects
+			(font
+				(size 0.381 0.381)
+			)
+			(justify left bottom)
+		)
+	)
+	(label "CODEC_OUT1P_1"
+		(at 163.83 77.47 0)
+		(effects
+			(font
+				(size 0.381 0.381)
+			)
+			(justify left bottom)
+		)
+	)
+	(label "CODEC_OUT1M_1"
+		(at 163.83 85.09 0)
+		(effects
+			(font
+				(size 0.381 0.381)
+			)
+			(justify left bottom)
+		)
+	)
+	(label "CODEC_OUT1M_2"
+		(at 176.53 85.09 0)
+		(effects
+			(font
+				(size 0.381 0.381)
+			)
+			(justify left bottom)
+		)
+	)
+	(label "CODEC_SPK1"
+		(at 220.98 82.55 0)
+		(effects
+			(font
+				(size 0.381 0.381)
+			)
+			(justify left bottom)
+		)
+	)
+	(label "CODEC_MEM_IN1P_1"
+		(at 59.69 80.01 0)
+		(effects
+			(font
+				(size 0.635 0.635)
+			)
+			(justify left bottom)
+		)
+	)
+	(label "CODEC_MEM_IN1M"
+		(at 86.36 82.55 0)
+		(effects
+			(font
+				(size 0.635 0.635)
+			)
+			(justify left bottom)
+		)
+	)
+	(label "CODEC_SPK2"
+		(at 220.98 80.01 0)
+		(effects
+			(font
+				(size 0.381 0.381)
+			)
+			(justify left bottom)
+		)
+	)
+	(label "CODEC_MEM_IN1M_1"
+		(at 59.69 82.55 0)
+		(effects
+			(font
+				(size 0.635 0.635)
+			)
+			(justify left bottom)
+		)
+	)
+	(label "CODEC_MEM_IN1P"
+		(at 86.36 80.01 0)
+		(effects
+			(font
+				(size 0.635 0.635)
+			)
+			(justify left bottom)
 		)
 	)
@@
 	(symbol
 		(lib_id "Device:C")
-		(at 161.29 77.47 90)
+		(at 160.02 77.47 90)
 		(unit 1)
 		(body_style 1)
@@
 		(fields_autoplaced yes)
 		(property "Reference" "C76"
-			(at 161.29 69.85 90)
+			(at 160.02 69.85 90)
 			(show_name no)
 			(do_not_autoplace no)
@@
 		)
 		(property "Value" "100n"
-			(at 161.29 72.39 90)
+			(at 160.02 72.39 90)
 			(show_name no)
 			(do_not_autoplace no)
@@
 		)
 		(property "Footprint" "Capacitor_SMD:C_0603_1608Metric"
-			(at 165.1 76.5048 0)
+			(at 163.83 76.5048 0)
 			(hide yes)
 			(show_name no)
@@
 		)
 		(property "Datasheet" ""
-			(at 161.29 77.47 0)
+			(at 160.02 77.47 0)
 			(hide yes)
 			(show_name no)
@@
 		)
 		(property "Description" "Unpolarized capacitor"
-			(at 161.29 77.47 0)
+			(at 160.02 77.47 0)
 			(hide yes)
 			(show_name no)
@@
 	(symbol
 		(lib_id "Device:C")
-		(at 161.29 85.09 270)
+		(at 160.02 85.09 270)
 		(mirror x)
 		(unit 1)
@@
 		(dnp no)
 		(property "Reference" "C77"
-			(at 161.29 92.71 90)
+			(at 160.02 92.71 90)
 			(show_name no)
 			(do_not_autoplace no)
@@
 		)
 		(property "Value" "100n"
-			(at 161.29 90.17 90)
+			(at 160.02 90.17 90)
 			(show_name no)
 			(do_not_autoplace no)
@@
 		)
 		(property "Footprint" "Capacitor_SMD:C_0603_1608Metric"
-			(at 157.48 84.1248 0)
+			(at 156.21 84.1248 0)
 			(hide yes)
 			(show_name no)
@@
 		)
 		(property "Datasheet" ""
-			(at 161.29 85.09 0)
+			(at 160.02 85.09 0)
 			(hide yes)
 			(show_name no)
@@
 		)
 		(property "Description" "Unpolarized capacitor"
-			(at 161.29 85.09 0)
-			(hide yes)
-			(show_name no)
+			(at 160.02 85.09 0)
+			(hide yes)
+			(show_name no)
