File: hardware/drone/drone.kicad_pcb (KiCad board)
At the start: 2 copper layers, 83 parts, among them J1 54548-2272, J2 BM08B-SRSS-TB_LF__SN_, J4 Conn_ARM_SWD_TagConnect_TC2030, Q1 ISP650P06NM, U1 STM32N645I0, U10 PE4259, U11 TAC5111IRGER, U12 LM4670SD/NOPB, U13 LP5907, U14 ICM-42688-P, U15 SAM_M10Q, U16 LMR51635XFDDCR, U17 TXU0204, U18 TPS2121, U19 BMP581, U2 SX1262IMLTRT, U20 TVS0500DRV, U21 TCA9406DC, U22 LIS2MDL, U23 MM8030_2610RJ3, U24 MM8030_2610RJ3, U25 ECMF2-40A100N6, U26 ECMF2-40A100N6, U27 ECMF2-40A100N6, U3 TPS628303, U4 TPS7A2118PQWDSGRQ1, U5 TPS628303, U6 MX25UW25645GXDI00, U7 CC3350, U8 DPX167125DT-8197B1, U9 DEA162450BT-1295A1

Commit message: More footprints
Parts:
- removed U12: LM4670SD/NOPB, Package_SON:WSON-8-1EP_3x3mm_P0.5mm_EP1.6x2.0mm
- added C1: 10n, Capacitor_SMD:C_0402_1005Metric, F.Cu at (161.0, 145.5)
- added C10: 1u, Capacitor_SMD:C_0201_0603Metric, F.Cu at (143.5, 107.6)
- added C100: 100n, Capacitor_SMD:C_0201_0603Metric, F.Cu at (164.8, 125.6)
- added C101: 100n, Capacitor_SMD:C_0201_0603Metric, F.Cu at (164.8, 127.3)
- added C102: 100n, Capacitor_SMD:C_0201_0603Metric, F.Cu at (164.8, 129.1)
- added C103: 100n, Capacitor_SMD:C_0201_0603Metric, F.Cu at (164.8, 130.8)
- added C104: 100n, Capacitor_SMD:C_0201_0603Metric, F.Cu at (167.2, 123.8)
- added C105: 1u, Capacitor_SMD:C_0201_0603Metric, F.Cu at (167.2, 125.6)
- added C106: 100n, Capacitor_SMD:C_0201_0603Metric, F.Cu at (167.2, 127.3)
- added C107: 100n, Capacitor_SMD:C_0201_0603Metric, F.Cu at (167.2, 129.1)
- added C108: 100n, Capacitor_SMD:C_0201_0603Metric, F.Cu at (167.2, 130.8)
- added C109: 1u, Capacitor_SMD:C_0201_0603Metric, F.Cu at (68.8, 145.1)
- added C110: 1u, Capacitor_SMD:C_0201_0603Metric, F.Cu at (68.8, 146.9)
- added C111: 1u, Capacitor_SMD:C_0201_0603Metric, F.Cu at (68.8, 148.6)
- added C112: 1u, Capacitor_SMD:C_0201_0603Metric, F.Cu at (68.8, 150.4)
- added C113: 1u, Capacitor_SMD:C_0201_0603Metric, F.Cu at (68.8, 152.1)
- added C114: 2.2u, Capacitor_SMD:C_1206_3216Metric, F.Cu at (111.2, 66.1)
- added C115: 1u, Capacitor_SMD:C_0201_0603Metric, F.Cu at (68.8, 153.9)
- added C116: 100n, Capacitor_SMD:C_0402_1005Metric, F.Cu at (167.0, 141.0)
- added C117: 100n, Capacitor_SMD:C_0402_1005Metric, F.Cu at (167.0, 143.0)
- added C118: 220n, Capacitor_SMD:C_0603_1608Metric, F.Cu at (161.5, 141.3)
- added C125: 100n, Capacitor_SMD:C_0603_1608Metric, F.Cu at (116.1, 64.8)
- added C126: 22u, Capacitor_SMD:CP_Elec_6.3x5.4, F.Cu at (118.8, 52.2)
- added C13: 4.7u, Capacitor_SMD:C_0603_1608Metric, F.Cu at (140.3, 100.3)
- added C14: 22u, Capacitor_SMD:C_0603_1608Metric, F.Cu at (140.3, 102.8)
- added C15: 22u, Capacitor_SMD:C_0603_1608Metric, F.Cu at (140.3, 105.3)
- added C17: 1u, Capacitor_SMD:C_0603_1608Metric, F.Cu at (161.5, 134.3)
- added C18: 1u, Capacitor_SMD:C_0603_1608Metric, F.Cu at (161.5, 136.8)
- added C2: 15u, Capacitor_SMD:C_0603_1608Metric, F.Cu at (161.5, 124.2)
- added C21: 4.7u, Capacitor_SMD:C_0402_1005Metric, F.Cu at (143.7, 104.0)
- added C24: 1u, Capacitor_SMD:C_0201_0603Metric, F.Cu at (68.8, 143.4)
- added C26: 4.7u, Capacitor_SMD:C_0603_1608Metric, F.Cu at (140.3, 107.8)
- added C27: 22u, Capacitor_SMD:C_0603_1608Metric, F.Cu at (140.3, 110.3)
- added C28: 22u, Capacitor_SMD:C_0603_1608Metric, F.Cu at (140.3, 112.8)
- added C29: 4.7u, Capacitor_SMD:C_0603_1608Metric, F.Cu at (149.1, 100.3)
- added C3: 15u, Capacitor_SMD:C_0603_1608Metric, F.Cu at (161.5, 126.7)
- added C30: 4.7u, Capacitor_SMD:C_0603_1608Metric, F.Cu at (149.1, 102.8)
- added C31: 4.7u, Capacitor_SMD:C_0603_1608Metric, F.Cu at (149.1, 105.3)
- added C4: 15u, Capacitor_SMD:C_0603_1608Metric, F.Cu at (161.5, 129.2)
- added C45: C, Capacitor_SMD:C_0402_1005Metric, F.Cu at (148.6, 109.5)
- added C5: 15u, Capacitor_SMD:C_0603_1608Metric, F.Cu at (161.5, 131.8)
- added C59: C, Capacitor_SMD:C_0402_1005Metric, F.Cu at (148.6, 113.5)
- added C6: 2.2n, Capacitor_SMD:C_0402_1005Metric, F.Cu at (165.0, 132.7)
- added C60: C, Capacitor_SMD:C_0402_1005Metric, F.Cu at (148.6, 115.5)
- added C66: 100n, Capacitor_SMD:C_0402_1005Metric, F.Cu at (154.5, 136.0)
- added C67: 10u, Capacitor_SMD:C_0805_2012Metric, F.Cu at (155.3, 124.5)
- added C68: 1u, Capacitor_SMD:C_0603_1608Metric, F.Cu at (151.1, 124.2)
- added C69: 10u, Capacitor_SMD:C_0805_2012Metric, F.Cu at (155.3, 127.5)
- added C7: 10u, Capacitor_SMD:C_0402_1005Metric, F.Cu at (143.7, 100.0)
- added C70: 100n, Capacitor_SMD:C_0402_1005Metric, F.Cu at (154.5, 138.0)
- added C71: 100n, Capacitor_SMD:C_0402_1005Metric, F.Cu at (154.5, 139.9)
- added C72: 10u, Capacitor_SMD:C_0805_2012Metric, F.Cu at (155.3, 130.5)
- added C73: 1u, Capacitor_SMD:C_0603_1608Metric, F.Cu at (151.1, 126.7)
- added C74: 1u, Capacitor_SMD:C_0603_1608Metric, F.Cu at (151.1, 129.2)
- added C75: 100n, Capacitor_SMD:C_0402_1005Metric, F.Cu at (154.5, 141.9)
- added C76: 100n, Capacitor_SMD:C_0603_1608Metric, F.Cu at (151.1, 131.8)
- added C77: 100n, Capacitor_SMD:C_0603_1608Metric, F.Cu at (151.1, 134.3)
- added C78: 1u, Capacitor_SMD:C_0603_1608Metric, F.Cu at (151.1, 136.8)
- added C79: 10u, Capacitor_SMD:C_0805_2012Metric, F.Cu at (155.3, 133.5)
- added C8: 10u, Capacitor_SMD:C_0402_1005Metric, F.Cu at (143.7, 102.0)
- added C80: 1u, Capacitor_SMD:C_0603_1608Metric, F.Cu at (71.4, 143.5)
- added C81: 1u, Capacitor_SMD:C_0603_1608Metric, F.Cu at (71.4, 145.5)
- added C85: 2.2u, Capacitor_SMD:C_1206_3216Metric, F.Cu at (111.2, 62.8)
- added C86: 100n, Capacitor_SMD:C_0603_1608Metric, F.Cu at (116.1, 62.3)
- added C87: 33u, Capacitor_SMD:C_1812_4532Metric, F.Cu at (104.9, 55.4)
- added C88: 33u, Capacitor_SMD:C_1812_4532Metric, F.Cu at (104.9, 60.4)
- added C89: 100n, Capacitor_SMD:C_0603_1608Metric, F.Cu at (74.9, 143.8)
- added C9: 1u, Capacitor_SMD:C_0201_0603Metric, F.Cu at (143.5, 105.8)
- added C92: 100n, Capacitor_SMD:C_0603_1608Metric, F.Cu at (167.9, 64.2)
- added C93: 10u, Capacitor_SMD:C_0805_2012Metric, F.Cu at (81.1, 144.0)
- added C94: 100n, Capacitor_SMD:C_0402_1005Metric, F.Cu at (80.3, 146.5)
- added C95: 47u, Capacitor_SMD:C_1206_3216Metric, F.Cu at (72.8, 150.1)
- added C96: 100n, Capacitor_SMD:C_0603_1608Metric, F.Cu at (74.9, 146.3)
- added C97: 100n, Capacitor_SMD:C_0603_1608Metric, F.Cu at (151.1, 139.3)
- added C98: 1u, Capacitor_SMD:C_0402_1005Metric, F.Cu at (71.4, 147.4)
- added C99: 100n, Capacitor_SMD:C_0201_0603Metric, F.Cu at (164.8, 123.8)
- added D3: TPD1E1B04DPYR, SoftDroneLibrary:TPD1E1B04DPYR, F.Cu at (174.8, 113.2)
- added D4: TPD1E1B04DPYR, SoftDroneLibrary:TPD1E1B04DPYR, F.Cu at (174.8, 115.0)
- added D5: B5819WS, Diode_SMD:D_SOD-323, F.Cu at (193.8, 97.5)
- added D6: TPD1E1B04DPYR, SoftDroneLibrary:TPD1E1B04DPYR, F.Cu at (170.2, 113.2)
- added D7: TPD1E1B04DPYR, SoftDroneLibrary:TPD1E1B04DPYR, F.Cu at (170.2, 115.0)
- added D8: TPD1E1B04DPYR, SoftDroneLibrary:TPD1E1B04DPYR, F.Cu at (170.2, 117.0)
- added D9: TPD1E1B04DPYR, SoftDroneLibrary:TPD1E1B04DPYR, F.Cu at (170.2, 118.8)
- added F1: 2920L150/60MR, Fuse:Fuse_2920_7451Metric, F.Cu at (179.1, 95.9)
- added FB1: 18R, Resistor_SMD:R_0603_1608Metric, F.Cu at (163.3, 101.1)
- added FB2: 120R, Resistor_SMD:R_0402_1005Metric, F.Cu at (163.0, 105.2)
- added J3: USB_C_Receptacle_USB2.0_16P, Connector_USB:USB_C_Receptacle_HRO_TYPE-C-31-M-12, F.Cu at (199.3, 116.7)
- added J5: Conn_01x06_Pin, Connector_PinHeader_2.54mm:PinHeader_1x06_P2.54mm_Vertical, F.Cu at (189.1, 113.2)
- added J6: Conn_01x02_Socket, Connector_JST:JST_SH_BM02B-SRSS-TB_1x02-1MP_P1.00mm_Vertical, F.Cu at (135.2, 78.5)
- added L12: L, Inductor_SMD:L_0402_1005Metric, F.Cu at (139.2, 65.0)
- added L4: L, Inductor_SMD:L_0402_1005Metric, F.Cu at (134.3, 65.0)
- added L5: L, Inductor_SMD:L_0402_1005Metric, F.Cu at (134.3, 67.0)
- added R1: 523k, Resistor_SMD:R_0402_1005Metric, F.Cu at (167.4, 76.0)
- added R10: 150k, Resistor_SMD:R_0603_1608Metric, F.Cu at (151.1, 144.3)
- added R11: 100k, Resistor_SMD:R_0402_1005Metric, F.Cu at (167.4, 84.0)
- added R12: 100k, Resistor_SMD:R_0402_1005Metric, F.Cu at (170.3, 76.0)
- added R13: 2.2k, Resistor_SMD:R_0402_1005Metric, F.Cu at (171.4, 69.9)
- added R14: 2.2k, Resistor_SMD:R_0402_1005Metric, F.Cu at (171.4, 71.9)
- added R15: 53.6k, Resistor_SMD:R_0603_1608Metric, F.Cu at (176.7, 76.3)
- added R16: 10.2k, Resistor_SMD:R_0603_1608Metric, F.Cu at (176.7, 78.8)
- added R17: 51.1k, Resistor_SMD:R_0402_1005Metric, F.Cu at (170.3, 78.0)
- added R18: 10.2k, Resistor_SMD:R_0402_1005Metric, F.Cu at (170.3, 80.0)
- added R19: 5k, Resistor_SMD:R_0402_1005Metric, F.Cu at (170.3, 82.0)
- added R2: 200k, Resistor_SMD:R_0402_1005Metric, F.Cu at (167.4, 78.0)
- added R20: 23.7k, Resistor_SMD:R_0402_1005Metric, F.Cu at (170.3, 84.0)
- added R21: 5k, Resistor_SMD:R_0402_1005Metric, F.Cu at (173.2, 76.0)
- added R22: 23.7k, Resistor_SMD:R_0402_1005Metric, F.Cu at (173.2, 78.0)
- added R23: 5k, Resistor_SMD:R_0402_1005Metric, F.Cu at (173.2, 80.0)
- added R24: 22k, Resistor_SMD:R_0603_1608Metric, F.Cu at (176.7, 81.3)
- added R25: 49.9k, Resistor_SMD:R_0603_1608Metric, F.Cu at (167.9, 66.7)
- added R26: 49.9k, Resistor_SMD:R_0603_1608Metric, F.Cu at (167.9, 69.2)
- added R27: 2.49k, Resistor_SMD:R_0603_1608Metric, F.Cu at (167.9, 71.8)
- added R28: 5.1k, Resistor_SMD:R_0402_1005Metric, F.Cu at (174.3, 64.0)
- added R29: 5.1k, Resistor_SMD:R_0402_1005Metric, F.Cu at (174.3, 66.0)
- added R3: 1.12M, Resistor_SMD:R_0402_1005Metric, F.Cu at (167.4, 80.0)
- added R30: 200R, Resistor_SMD:R_0402_1005Metric, F.Cu at (174.3, 68.0)
- added R31: 200R, Resistor_SMD:R_0402_1005Metric, F.Cu at (174.3, 69.9)
- added R32: 10k, Resistor_SMD:R_0402_1005Metric, F.Cu at (174.3, 71.9)
- added R33: 10k, Resistor_SMD:R_0402_1005Metric, F.Cu at (177.2, 64.0)
- added R34: 200R, Resistor_SMD:R_0402_1005Metric, F.Cu at (186.1, 64.0)
- added R35: 47k, Resistor_SMD:R_0402_1005Metric, F.Cu at (182.1, 76.0)
- added R36: 47k, Resistor_SMD:R_0402_1005Metric, F.Cu at (182.1, 78.0)
- added R37: 47k, Resistor_SMD:R_0402_1005Metric, F.Cu at (182.1, 80.0)
- added R38: 47k, Resistor_SMD:R_0402_1005Metric, F.Cu at (182.1, 82.0)
- added R39: 47k, Resistor_SMD:R_0402_1005Metric, F.Cu at (182.1, 84.0)
- added R4: 200k, Resistor_SMD:R_0402_1005Metric, F.Cu at (167.4, 82.0)
- added R40: 10K, Resistor_SMD:R_0402_1005Metric, F.Cu at (177.2, 66.0)
- added R41: R, Resistor_SMD:R_0603_1608Metric, F.Cu at (182.7, 64.2)
- added R42: R, Resistor_SMD:R_0603_1608Metric, F.Cu at (182.7, 66.7)
- added R43: 2.2k, Resistor_SMD:R_0402_1005Metric, F.Cu at (177.2, 68.0)
- added R44: 2.2k, Resistor_SMD:R_0402_1005Metric, F.Cu at (177.2, 69.9)
- added R45: 2R, Resistor_SMD:R_0402_1005Metric, F.Cu at (173.2, 82.0)
- added R5: 10K, Resistor_SMD:R_0402_1005Metric, F.Cu at (171.4, 64.0)
- added R6: 10K, Resistor_SMD:R_0402_1005Metric, F.Cu at (171.4, 66.0)
- added R7: 10K, Resistor_SMD:R_0402_1005Metric, F.Cu at (171.4, 68.0)
- added R8: 100R, Resistor_SMD:R_0402_1005Metric, F.Cu at (139.2, 67.0)
- added R9: 150k, Resistor_SMD:R_0603_1608Metric, F.Cu at (151.1, 141.8)
- added U28: LM4670ITL/NOPB, LM4670ITL_NOPB:BGA9C50P3X3_146X148X68, F.Cu at (91.4, 63.6)
- C119, C121: footprint Capacitor_SMD:C_0201_0603Metric -> Capacitor_SMD:C_0603_1608Metric
- moved J2 12.1 mm to (84.2, 54.0)
- moved U7 6.00 mm to (75.5, 100.2)

Commit message: Completed footprint assignments
Parts:
- removed U13: LP5907, LP5907A28YKMR:BGA4C35P2X2_64X64X50
- added AE2: Antenna, ANT-916-HETH:ANT916HETH, F.Cu at (136.6, 47.1)
- added C122: 20p, Capacitor_SMD:C_0201_0603Metric, F.Cu at (209.9, 99.3)
- added C43: C, Capacitor_SMD:C_0201_0603Metric, F.Cu at (214.3, 94.1)
- added C44: C, Capacitor_SMD:C_0201_0603Metric, F.Cu at (214.3, 95.8)
- added C58: 20p, Capacitor_SMD:C_0201_0603Metric, F.Cu at (209.9, 94.1)
- added C62: C, Capacitor_SMD:C_0201_0603Metric, F.Cu at (209.9, 95.8)
- added C63: C, Capacitor_SMD:C_0201_0603Metric, F.Cu at (209.9, 97.6)
- added D1: MM3Z10, Diode_SMD:D_SOD-323, F.Cu at (197.4, 84.0)
- added D2: SMBJ30CA, Diode_SMD:D_SMB, F.Cu at (199.5, 79.8)
- added L1: 1u, SoftDroneLibrary:CVH201610A-2R2M, F.Cu at (222.4, 82.7)
- added L10: 15n, Inductor_SMD:L_0402_1005Metric, F.Cu at (212.8, 88.0)
- added L11: 15u, Inductor_SMD:L_0603_1608Metric, F.Cu at (222.2, 87.9)
- added L13: 10u, SoftDroneLibrary:CYA0650-10UH, F.Cu at (109.8, 42.9)
- added L2: 0.47u, SoftDroneLibrary:TFM201610ALC-R47MTAA, F.Cu at (110.7, 122.0)
- added L3: 0.47u, SoftDroneLibrary:TFM201610ALC-R47MTAA, F.Cu at (105.6, 128.3)
- added L6: 0R, Inductor_SMD:L_0402_1005Metric, F.Cu at (212.8, 80.0)
- added L7: 47n, Inductor_SMD:L_0402_1005Metric, F.Cu at (212.8, 82.0)
- added L8: 2.5n, Inductor_SMD:L_0402_1005Metric, F.Cu at (212.8, 84.0)
- added L9: 4.7n, Inductor_SMD:L_0402_1005Metric, F.Cu at (212.8, 86.0)
- added SW1: SW_MEC_5E, SoftDroneLibrary:1825910-6, F.Cu at (99.5, 153.5)
- added U12: LP5907, LP5907A28YKMR:BGA4C35P2X2_64X64X50, F.Cu at (91.7, 72.1)
- added Y1: Crystal_GND24, Crystal:Crystal_SMD_3225-4Pin_3.2x2.5mm, F.Cu at (30.7, 55.5)
- added Y2: Crystal_GND24, Crystal:Crystal_SMD_3225-4Pin_3.2x2.5mm, F.Cu at (30.7, 62.0)
- added Y3: Crystal_GND24, SoftDroneLibrary:XTM32048000NT00351001, F.Cu at (36.0, 50.3)
- added Y4: Crystal, SoftDroneLibrary:FC-135R 32.7680KA-A3, F.Cu at (26.5, 72.9)

Commit message: Added chip antenna footprint
Parts:
- added AE1: Antenna, SoftDroneLibrary:ANT-DB1-NSP250-T, F.Cu at (177.1, 49.7)
- C43, C44: value C -> 20p
- C62, C63: value C -> 10p
Changed lines of the file:
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@@
 			)
 		)
-		(property "Value" "C"
+		(property "Value" "10p"
 			(at 0 1.05 0)
 			(layer "F.Fab")
@@
 			)
 		)
-		(property "Value" "C"
+		(property "Value" "20p"
 			(at 0 1.05 0)
 			(layer "F.Fab")
@@
 			)
 		)
-		(property "Value" "C"
+		(property "Value" "10p"
 			(at 0 1.05 0)
 			(layer "F.Fab")
@@
 		)
 	)
+	(footprint "SoftDroneLibrary:ANT-DB1-NSP250-T"
+		(layer "F.Cu")
+		(at 177.115 49.725)
+		(property "Reference" "AE1"
+			(at -0.02 -18.25 0)
+			(unlocked yes)
+			(layer "F.SilkS")
+			(effects
+				(font
+					(size 1 1)
+					(thickness 0.1)
+				)
+			)
+		)
+		(property "Value" "Antenna"
+			(at -0.02 -16.75 0)
+			(unlocked yes)
+			(layer "F.Fab")
+			(effects
+				(font
+					(size 1 1)
+					(thickness 0.15)
+				)
+			)
+		)
+		(property "Datasheet" ""
+			(at 0 0 0)
+			(unlocked yes)
+			(layer "F.Fab")
+			(hide yes)
+			(effects
+				(font
+					(size 1 1)
+					(thickness 0.15)
+				)
+			)
+		)
+		(property "Description" "Antenna"
+			(at 0 0 0)
+			(unlocked yes)
+			(layer "F.Fab")
+			(hide yes)
+			(effects
+				(font
+					(size 1 1)
+					(thickness 0.15)
+				)
+			)
+		)
+		(sheetname "/RF_5GHz/")
+		(sheetfile "rf_5ghz.kicad_sch")
+		(units
+			(unit
+				(name "A")
+				(pins "1")
+			)
+		)
+		(attr smd)
+		(duplicate_pad_numbers_are_jumpers no)
+		(fp_line
+			(start -3.65 1.7)
+			(end 5.93 1.7)
+			(stroke
+				(width 0.1)
+				(type default)
+			)
+			(layer "F.SilkS")
+		)
+		(fp_rect
+			(start -4.19 -8.35)
+			(end 6.19 1.94)
+			(stroke
+				(width 0.1)
+				(type solid)
+			)
+			(fill no)
+			(layer "F.CrtYd")
+		)
+		(fp_text user "${REFERENCE}"
+			(at -0.02 -15.25 0)
+			(unlocked yes)
+			(layer "F.Fab")
+			(effects
+				(font
+					(size 1 1)
+					(thickness 0.15)
+				)
+			)
+		)
+		(pad "1" smd roundrect
+			(at -2.54 0)
+			(size 2.24 2.74)
+			(layers "F.Cu" "F.Mask" "F.Paste")
+			(roundrect_rratio 0.03)
+			(net "/RF_5GHz/CC_ANT_FEED")
+			(pinfunction "A_1")
+			(pintype "input")
+		)
+		(pad "2" smd roundrect
+			(at 2.54 0)
+			(size 2.24 2.74)
+			(layers "F.Cu" "F.Mask" "F.Paste")
+			(roundrect_rratio 0.03)
+		)
+		(embedded_fonts no)
+		(model "/home/alexshort/Repos/drone/hardware/Components/LIB_ANT-DB1-NSP250-T/ANT-DB1-NSP250-T/3D/ANT-DB1-NSP250-T.stp"
+			(offset
+				(xyz 1 -1.25 0)
+			)
+			(scale
+				(xyz 1 1 1)
+			)
+			(rotate
+				(xyz -90 -0 -0)
+			)
+		)
+	)
 	(footprint "Capacitor_SMD:C_0201_0603Metric"
 		(layer "F.Cu")
@@
 			)
 		)
-		(property "Value" "C"
+		(property "Value" "20p"
 			(at 0 1.05 0)
 			(layer "F.Fab")

Commit message: Labeled nets, added colours, and fixed stm32n6 schematic symbol issues
Parts:
- added C127: 100n, Capacitor_SMD:C_0201_0603Metric, F.Cu at (69.0, 42.4)
- moved U1 40.1 mm to (81.0, 32.8)
Connections:
- net /RF_5GHz/CC_ANT_FEED renamed /RF_5GHz/RF5G_ANT
- net /RF_5GHz/RF_A renamed /RF_5GHz/RF5G_A
- net /RF_5GHz/RF_BG renamed /RF_5GHz/RF5G_BG
- net Net-(AE2-A) renamed /RF_915/RFCSUBG_ANT
- net Net-(C48-Pad1) renamed /RF_915/RFOSUBG_2
- net Net-(C48-Pad2) renamed /RF_915/RFOSUBG_3
- net Net-(C51-Pad2) renamed /RF_915/RFOSUBG_4
- net Net-(C76-Pad2) renamed /Audio/CODEC_OUT1P_1
- net Net-(C77-Pad1) renamed /Audio/CODEC_OUT1M_1
- net Net-(D1-A) renamed /Power/VBAT_PMOS_G
- net Net-(D2-A2) renamed /Power/VBAT_PMOS_D
- net Net-(D3-A2) renamed /MCU/USBC_D-
- net Net-(D4-A2) renamed /MCU/USBC_D+
- net Net-(D5-A) renamed /MCU/OSPI_NRESET_CHIP
- net Net-(J3-CC1) renamed /MCU/USBC_CC1
- net Net-(J3-CC2) renamed /MCU/USBC_CC2
- net Net-(J6-Pin_1) renamed /Audio/CODEC_SPK1
- net Net-(J6-Pin_2) renamed /Audio/CODEC_SPK2
- net Net-(L1-Pad2) renamed /Power/MCU_VLXSMPS
- net Net-(MK2-OUT+) renamed /Audio/CODEC_MEM_IN1P_1
- net Net-(MK2-OUT-) renamed /Audio/CODEC_MEM_IN1M_1
- net Net-(U10-CTRL) renamed /RF_915/SX_SW_CTRL
- net Net-(U10-RF1) renamed /RF_915/RFOSUBG_5
- net Net-(U10-RF2) renamed /RF_915/RFISUBG_3
- net Net-(U10-RFC) renamed /RF_915/RFCSUBG_1
- net Net-(U11-IN1M) renamed /Audio/CODEC_MEM_IN1M
- net Net-(U11-IN1P) renamed /Audio/CODEC_MEM_IN1P
- net Net-(U11-OUT1M) renamed /Audio/CODEC_OUT1M
- net Net-(U11-OUT1P) renamed /Audio/CODEC_OUT1P
- net Net-(U16-FB) renamed /Power/VSYS_5V_FB
- net Net-(U16-SW) renamed /Power/VSYS_5V_SW
- net Net-(U18-ILM) renamed /Power/PMUX_ILM
- net Net-(U18-SS) renamed /Power/PMUX_SS
- net Net-(U1CSI-CSI_REXT) renamed /Camera/CSI_REXT
- net Net-(U1PA-PA12) renamed /MCU/MCU_PA12_ADC
- net Net-(U1PC-PC14-OSC32_IN) renamed /MCU/MCU_LF_OSC_IN
- net Net-(U1PC-PC15-OSC32_OUT) renamed /MCU/MCU_LF_OSC_OUT
- net Net-(U1Power-V08CAP) renamed /Power/MCU_V08CAP
- net Net-(U1USB-OTG1_TXRTUNE) renamed /MCU/OTG1_TXRTUNE
- net Net-(U1USB-OTG2_TXRTUNE) renamed /MCU/OTG2_TXRTUNE
- net Net-(U2-RFI_N) renamed /RF_915/RFISUBG_1
- net Net-(U2-RFI_P) renamed /RF_915/RFISUBG_2
- net Net-(U2-RFO) renamed /RF_915/RFOSUBG_1
- net Net-(U2-VR_PA) renamed /RF_915/RFVRSUBG
- net Net-(U2-XTA) renamed /RF_915/SX_XTA
- net Net-(U2-XTB) renamed /RF_915/SX_XTB
- net Net-(U23-IN) renamed /RF_5GHz/RF5G_1
- net Net-(U23-OUT) renamed /RF_5GHz/RF5G_2
- net Net-(U24-OUT) renamed /RF_915/RFCSUBG_2
- net Net-(U28-+IN) renamed /Audio/CODEC_OUT1M_2
- net Net-(U28--IN) renamed /Audio/CODEC_OUT1P_2
- net Net-(U3-FB) renamed /Power/VDD1V8_FB
- net Net-(U3-SW) renamed /Power/VDD1V8_SW
- net Net-(U5-FB) renamed /Power/VDD3V3_FB
- net Net-(U5-SW) renamed /Power/VDD3V3_SW
- net Net-(U6-~{ECS}) renamed /MCU/OSPI_NECS
- net Net-(U7-HFXT_M) renamed /RF_5GHz/CC_HFXT_M
- net Net-(U7-HFXT_P/EXT) renamed /RF_5GHz/CC_HFXT_P
- net Net-(U8-Low-Band_Port) renamed /RF_5GHz/RF5G_BG_1
- R32 pad 1: Net-(U1MISC-BOOT0) -> /MCU/MCU_BOOT0
- R33 pad 1: Net-(U1PA-PA6) -> /MCU/MCU_BOOT0
- U1 pad D3: Net-(U1MISC-BOOT0) -> /MCU/MCU_BOOT0
- U1 pad E2: (no net) -> GND
- U1 pad L4: (no net) -> VDD1V8
- U1 pad L8: Net-(U1PA-PA6) -> /MCU/MCU_BOOT0
- U1 pad M12: (no net) -> unconnected-(U1PG-PG0-PadM12)
- U1 pad M9: (no net) -> unconnected-(U1PG-PG1-PadM9)

Commit message: Started layout and tested RF routing paths
Parts:
- C45, C59, C60: footprint Capacitor_SMD:C_0402_1005Metric -> Capacitor_SMD:C_0603_1608Metric
- J1, U1, U6: moved to B.Cu
- L12, L4, L5: footprint Inductor_SMD:L_0402_1005Metric -> Inductor_SMD:L_0603_1608Metric
- moved U10 149.2 mm to (193.5, 125.6)
- moved U1 137.3 mm to (195.2, 109.0), turned to 90 degrees
- moved U8 130.0 mm to (191.4, 95.8), turned to -90 degrees
- moved U2 126.7 mm to (178.4, 126.3), turned to -90 degrees
- moved J1 124.4 mm to (173.5, 109.5), turned to 90 degrees
- moved C34 123.8 mm to (185.3, 253.9)
- moved C83 123.8 mm to (187.6, 269.0)
- moved C31 123.8 mm to (201.5, 217.5)
- moved D4 123.8 mm to (227.1, 227.2)
- moved L1 123.8 mm to (274.7, 194.8)
- moved R23 123.8 mm to (225.6, 192.2)
- moved R42 123.8 mm to (235.0, 178.9)
- moved R6 123.8 mm to (223.7, 178.1)
- moved R7 123.8 mm to (223.7, 180.1)
- moved C109 123.8 mm to (121.1, 257.3)
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Connections:
- net Net-(U7-PA_LDO_OUT) renamed /RF_5GHz/CC_PA_LDO_OUT
Routing:
- net /RF_915/RFCSUBG_ANT: track 0.00 -> 11.6 mm
- net /RF_915/RFISUBG_3: track 0.00 -> 8.78 mm
- net /RF_5GHz/RF5G_BG_1: track 0.00 -> 4.22 mm
- net /RF_5GHz/RF5G_ANT: track 0.00 -> 4.12 mm
- net /RF_5GHz/RF5G_A: track 0.00 -> 3.46 mm
- net /RF_5GHz/RF5G_BG: track 0.00 -> 3.35 mm
- net /RF_915/RFOSUBG_2: track 0.00 -> 2.85 mm
- net /RF_915/RFOSUBG_3: track 0.00 -> 2.77 mm
- net /RF_5GHz/RF5G_2: track 0.00 -> 2.70 mm
- net /RF_915/RFCSUBG_2: track 0.00 -> 2.63 mm
- net /RF_915/RFISUBG_2: track 0.00 -> 2.55 mm
- net /RF_915/RFISUBG_1: track 0.00 -> 2.52 mm
- net VDD1V8: track 0.00 -> 2.26 mm, vias 0 -> 4
- net /RF_915/RFOSUBG_5: track 0.00 -> 2.14 mm
- net /RF_915/RFOSUBG_1: track 0.00 -> 1.70 mm
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Other:
- board outline added: 45 x 45 mm
- copper layers 2 -> 6
