File: hardware/drone/drone.kicad_pcb (KiCad board)
At the start: 6 copper layers, 45 x 45 mm, 244 parts, among them J1 54548-2272, J2 BM08B-SRSS-TB_LF__SN_, J3 USB_C_Receptacle_USB2.0_16P, J4 Conn_ARM_SWD_TagConnect_TC2030, J5 Conn_01x06_Pin, J6 Conn_01x02_Socket, SW1 SW_MEC_5E, U1 STM32N645I0, U10 PE4259, U11 TAC5111IRGER, U12 LP5907, U13 SQA411CEJW-T1_GE3, U14 ICM-42688-P, U15 SAM_M10Q, U16 LMR51635YFDDCR, U17 TXU0204, U18 TPS2121, U19 BMP581, U2 SX1262IMLTRT, U20 TVS0500DRV, U21 TCA9406DC, U22 LIS2MDL, U23 MM8030_2610RJ3, U24 MM8030_2610RJ3, U25 ECMF2-40A100N6, U26 ECMF2-40A100N6, U27 ECMF2-40A100N6, U28 LM4670ITL/NOPB, U3 TPS628303, U4 TPS7A2118PQWDSGRQ1, U5 TPS628303, U6 MX25UW25645GXDI00, U7 CC3350, U8 DPX167125DT-8197B1, U9 DEA162450BT-1295A1, Y1 Crystal_GND24, Y2 Crystal_GND24, Y3 Crystal_GND24, Y4 Crystal

Commit message: Changed layout and picked new drone chassis
Parts:
- U4: moved to B.Cu
- moved L12 213.0 mm to (415.2, 132.5)
- moved C59 213.0 mm to (413.0, 133.3)
- moved C60 213.0 mm to (417.4, 133.3)
- moved AE2 212.8 mm to (424.0, 132.5), turned to -90 degrees
- moved C48 206.9 mm to (393.4, 126.0)
- moved C50 206.9 mm to (394.8, 126.5)
- moved C52 206.9 mm to (399.4, 126.5)
- moved C54 206.9 mm to (391.5, 127.9)
- moved L6 206.9 mm to (390.5, 126.9)
- moved L8 206.9 mm to (393.4, 126.9)
- moved L9 206.9 mm to (398.0, 126.9)
- moved U10 206.9 mm to (401.7, 127.6)
- moved C46 206.9 mm to (390.1, 125.5)
- moved C47 206.9 mm to (391.0, 125.5)
- moved C51 206.9 mm to (396.2, 126.9)
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Routing:
- net /Camera/CSI_D1N: track 29.1 -> 0.00 mm, vias 1 -> 0
- net /Camera/CSI_D0N: track 28.7 -> 0.00 mm, vias 1 -> 0
- net /Camera/CSI_D1P: track 28.1 -> 0.00 mm, vias 1 -> 0
- net /Camera/CSI_D0P: track 27.7 -> 0.00 mm, vias 1 -> 0
- net /Camera/CSI_CKN: track 26.9 -> 0.00 mm, vias 1 -> 0
- net /Camera/CSI_CKP: track 25.9 -> 0.00 mm, vias 1 -> 0
- net /RF_5GHz/RF5G_2: track 2.70 -> 13.6 mm
- net /RF_915/RFCSUBG_2: track 2.63 -> 11.6 mm
- net /RF_915/RFCSUBG_ANT: track 1.42 -> 6.59 mm
Other:
- board size 45 x 45 mm -> 80 x 44 mm

Commit message: Placed connectors and bucks
Parts:
- D1, F1, J2, J3, U13: moved to F.Cu
- D2: value SMBJ30CA -> 6DFN36CA; footprint Diode_SMD:D_SMB -> SoftDroneLibrary:6DFN12CA
- R12: moved to B.Cu
- moved C89 326.7 mm to (444.0, 175.7)
- moved C95 276.3 mm to (381.6, 159.5)
- moved C96 272.3 mm to (381.6, 161.4)
- moved U20 250.5 mm to (382.4, 165.2)
- moved J1 221.7 mm to (401.0, 171.0), turned to 0 degrees
- moved R17 217.9 mm to (439.6, 170.1)
- moved U25 216.2 mm to (400.1, 165.9), turned to 0 degrees
- moved R12 214.9 mm to (437.4, 197.8)
- moved U27 212.7 mm to (398.2, 165.9), turned to 0 degrees
- moved U26 209.1 mm to (396.3, 165.9), turned to 0 degrees
- moved R15 205.6 mm to (378.1, 166.7), turned to -90 degrees
- moved U1 205.1 mm to (390.9, 148.1), turned to 180 degrees
- moved R16 202.9 mm to (376.6, 166.8), turned to 90 degrees
- moved C86 200.9 mm to (376.6, 163.9), turned to 90 degrees
- moved U16 197.6 mm to (374.1, 165.9), turned to 90 degrees
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Connections:
- J2 pad 2: unconnected-(J2-Pad2) -> VBAT_UNPROT
Routing:
- net /MCU/OSPI_IO3: track 7.94 -> 2.66 mm
- net /MCU/OSPI_DQS: track 12.7 -> 7.98 mm
- net /MCU/OSPI_IO5: track 9.50 -> 5.37 mm
- net /MCU/OSPI_IO0: track 14.3 -> 10.9 mm
- net /MCU/OSPI_IO7: track 9.69 -> 6.98 mm
- net /MCU/OSPI_IO2: track 8.16 -> 9.62 mm
- net /MCU/OSPI_IO6: track 8.06 -> 7.10 mm
- net /MCU/OSPI_IO4: track 8.23 -> 9.15 mm
Other:
- board size 80 x 44 mm -> 80 x 50 mm

Commit message: MCU decap placement and camera connector placement
Parts:
- moved C24 294.5 mm to (397.1, 152.7), turned to -90 degrees
- moved C112 294.1 mm to (392.9, 150.1)
- moved C111 291.6 mm to (391.3, 150.9), turned to -90 degrees
- moved C110 291.3 mm to (390.9, 148.9), turned to 90 degrees
- moved C109 289.2 mm to (389.7, 150.1), turned to 90 degrees
- moved U11 283.8 mm to (454.9, 148.9)
- moved C127 272.4 mm to (393.7, 151.7), turned to -90 degrees
- moved C23 244.0 mm to (397.8, 152.7), turned to -90 degrees
- moved C22 244.0 mm to (398.5, 152.7), turned to -90 degrees
- moved C20 240.8 mm to (395.5, 152.2), turned to -45 degrees
- moved C100 203.8 mm to (400.6, 149.2)
- moved C104 195.6 mm to (396.0, 151.7), turned to -45 degrees
- moved C105 195.0 mm to (395.0, 152.7), turned to -45 degrees
- moved C108 193.9 mm to (388.9, 148.5), turned to -90 degrees
- moved C107 193.8 mm to (388.9, 146.9), turned to 90 degrees
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Connections:
- net /Power/MCU_VLXSMPS renamed /Power/VLXSMPS
Routing:
- net /Camera/CSI_CKN: track 0.00 -> 16.1 mm, vias 0 -> 1
- net /Camera/CSI_D1N: track 0.00 -> 15.6 mm, vias 0 -> 1
- net /Camera/CSI_D0N: track 0.00 -> 15.4 mm, vias 0 -> 1
- net /Camera/CSI_CKP: track 0.00 -> 15.1 mm, vias 0 -> 1
- net /Camera/CSI_D1P: track 0.00 -> 14.6 mm, vias 0 -> 1
- net /Camera/CSI_D0P: track 0.00 -> 14.5 mm, vias 0 -> 1
- net GND: track 1.91 -> 13.7 mm, vias 4 -> 14
- net VDD1V8: track 2.26 -> 8.75 mm, vias 4 -> 6
- net VDDCORE: track 0.57 -> 4.02 mm, vias 1 -> 5
- net /Camera/CSI_CON_D0P: track 2.37 -> 0.00 mm
- net /Camera/CSI_CON_D0N: track 2.37 -> 0.00 mm
- net /Camera/CSI_CON_CKN: track 2.33 -> 0.00 mm
- net /Camera/CSI_CON_CKP: track 2.33 -> 0.00 mm
- net /Camera/CSI_CON_D1N: track 2.20 -> 0.00 mm
- net /Camera/CSI_CON_D1P: track 2.20 -> 0.00 mm
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
Commit message: More decap placement
Parts:
- C2, C3, C4, C5, L1: moved to B.Cu
- moved C12 239.7 mm to (394.9, 148.1), turned to 90 degrees
- moved C11 238.3 mm to (394.0, 148.1), turned to 90 degrees
- moved C10 213.0 mm to (396.4, 148.1), turned to 90 degrees
- moved C8 212.8 mm to (398.4, 148.1), turned to 90 degrees
- moved C9 211.7 mm to (395.6, 148.1), turned to 90 degrees
- moved C7 211.3 mm to (397.3, 148.1), turned to 90 degrees
- moved C3 210.9 mm to (402.8, 145.2)
- moved C4 210.3 mm to (400.4, 144.3), turned to 90 degrees
- moved C5 210.1 mm to (398.9, 144.3), turned to 90 degrees
- moved C2 209.1 mm to (402.8, 146.7)
- moved C101 195.8 mm to (389.7, 146.9), turned to -90 degrees
- moved C6 193.8 mm to (382.2, 143.1)
- moved R45 165.0 mm to (381.3, 139.6)
- moved L1 45.2 mm to (399.0, 147.7), turned to 180 degrees
- moved C100 9.63 mm to (391.3, 146.9)
Routing:
- net VDD1V8: track 8.75 -> 16.2 mm, vias 6 -> 11
- net GND: track 13.7 -> 19.2 mm, vias 14 -> 20
- net /Power/VLXSMPS: track 0.00 -> 2.89 mm

Commit message: Routed CC3350 RF, SDMMC, decoupling and crystal
Parts:
- R35, R36, R37, R38, R39: moved to B.Cu
- moved Y1 296.0 mm to (376.4, 128.0), turned to 90 degrees
- moved C37 226.2 mm to (375.5, 131.6)
- moved C36 225.7 mm to (375.5, 130.8)
- moved C38 224.9 mm to (370.6, 127.5)
- moved C39 221.9 mm to (370.6, 135.1), turned to 180 degrees
- moved C35 217.3 mm to (369.2, 135.1), turned to 180 degrees
- moved C42 213.8 mm to (367.4, 134.3), turned to -90 degrees
- moved R39 151.1 mm to (369.5, 128.2), turned to -90 degrees
- moved R38 151.1 mm to (370.4, 128.2), turned to -90 degrees
- moved R35 146.9 mm to (368.5, 128.2), turned to -90 degrees
- moved R37 146.2 mm to (367.9, 132.6)
- moved R36 145.7 mm to (367.9, 131.6)
- moved C44 134.7 mm to (374.2, 126.9), turned to 90 degrees
- moved C43 134.1 mm to (377.3, 130.4)
- moved U23 0.73 mm to (372.6, 140.6)
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Connections:
- net Net-(U7-DIG_LDO_OUT) renamed /RF_5GHz/CC_DIG_LDO_OUT
Routing:
- net CC_SDMMC1_CMD: track 0.57 -> 42.3 mm, vias 1 -> 2
- net CC_SDMMC1_D0: track 0.57 -> 38.6 mm, vias 1 -> 2
- net CC_SDMMC1_D1: track 0.57 -> 38.4 mm, vias 1 -> 2
- net CC_SDMMC1_CLK: track 0.57 -> 37.0 mm, vias 1 -> 2
- net CC_SDMMC1_D2: track 0.57 -> 36.0 mm, vias 1 -> 2
- net CC_SDMMC1_D3: track 0.57 -> 35.3 mm, vias 1 -> 2
- net GND: track 19.2 -> 26.7 mm, vias 20 -> 151
- net VDD1V8: track 16.2 -> 21.8 mm, vias 11 -> 16
- net /RF_5GHz/CC_HFXT_M: track 0.00 -> 5.48 mm
- net /RF_5GHz/CC_HFXT_P: track 0.00 -> 5.21 mm
- net /RF_5GHz/RF5G_ANT: track 1.43 -> 4.49 mm
- net CC_RESET: track 0.00 -> 0.86 mm, vias 0 -> 1
- net VDD3V3: vias 0 -> 2
- added copper zone on F.Cu, net /RF_5GHz/CC_DIG_LDO_OUT
- added copper zone on F.Cu, net GND
- added copper zone on F.Cu, net VDD1V8
- added copper zone on F.Cu, net VDD3V3

Commit message: More CC3350 routing
Parts:
- R35, R36, R37, R38, R39: footprint Resistor_SMD:R_0402_1005Metric -> Resistor_SMD:R_0201_0603Metric
- moved R45 28.3 mm to (386.6, 111.8)
- moved C6 28.3 mm to (387.6, 115.3)
- moved R37 5.44 mm to (370.9, 128.0), turned to -90 degrees
- moved R36 5.14 mm to (371.6, 128.0), turned to -90 degrees
- moved R35 0.32 mm to (368.8, 128.0)
- moved R38 0.30 mm to (370.2, 128.0)
- moved R39 0.21 mm to (369.5, 128.0)
Routing:
- net CC_SDMMC1_D0: track 38.6 -> 43.0 mm
- net /RF_5GHz/CC_LOGGER: track 0.00 -> 1.55 mm, vias 0 -> 1
- net /RF_5GHz/CC_SWDIO: track 0.00 -> 1.37 mm, vias 0 -> 1
- net CC_SDMMC1_CMD: track 42.3 -> 41.1 mm
- net /RF_5GHz/CC_SWCLK: track 0.00 -> 1.16 mm, vias 0 -> 1
- net CC_IRQ_WL: track 0.00 -> 1.14 mm, vias 0 -> 1
- net CC_SDMMC1_D1: track 38.4 -> 39.0 mm
- net GND: track 26.7 -> 26.1 mm, vias 151 -> 155

Commit message: SX1262 layout and decoupling
Parts:
- C57: footprint Capacitor_SMD:C_0402_1005Metric -> Capacitor_SMD:C_0201_0603Metric
- C64, C65: footprint Capacitor_SMD:C_0402_1005Metric -> Capacitor_SMD:C_0201_0603Metric; moved to B.Cu
- moved C57 230.8 mm to (386.4, 127.8), turned to 180 degrees
- moved C56 225.3 mm to (382.3, 129.6), turned to -90 degrees
- moved C65 221.7 mm to (383.4, 131.7)
- moved C64 221.1 mm to (383.4, 131.0)
- moved L11 127.9 mm to (381.1, 129.4), turned to 90 degrees
- moved C47 1.74 mm to (389.8, 128.0)
- moved C50 1.74 mm to (393.6, 129.0)
- moved C51 1.74 mm to (395.0, 129.4)
- moved C54 1.74 mm to (390.3, 130.3)
- moved L10 1.74 mm to (388.9, 130.8)
- moved L7 1.74 mm to (390.8, 128.9)
- moved C46 1.74 mm to (388.9, 128.0)
- moved C52 1.74 mm to (398.3, 128.9)
- moved L6 1.74 mm to (389.4, 129.4)
- moved L8 1.74 mm to (392.2, 129.4)
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Connections:
- net /RF_915/SX_DCC_SW renamed /RF_915/SX_SMPS_SW
Routing:
- net /Camera/CSI_D1N: track 15.6 -> 2.74 mm
- net /Camera/CSI_D1P: track 14.6 -> 1.76 mm
- net /Camera/CSI_CKP: track 15.1 -> 3.46 mm
- net /Camera/CSI_D0P: track 14.5 -> 2.85 mm
- net /Camera/CSI_D0N: track 15.4 -> 3.83 mm
- net /Camera/CSI_CKN: track 16.1 -> 4.66 mm
- net VDD3V3: track 0.00 -> 2.26 mm, vias 2 -> 3
- net /RF_915/RFCSUBG_ANT: track 6.59 -> 8.00 mm
- net VDD1V8: track 21.8 -> 23.0 mm, vias 16 -> 17
- net GND: track 26.1 -> 27.1 mm, vias 155 -> 181
- net /RF_915/RFCSUBG_2: track 11.6 -> 12.6 mm
- added copper zone on B.Cu, net GND
Other:
- outline, holes or cut-outs redrawn

Commit message: Routed CSI
Parts:
- moved Y2 304.4 mm to (383.6, 126.4)
- moved U25 1.83 mm to (398.8, 165.5)
- moved U26 1.83 mm to (395.0, 165.5)
- moved U27 1.83 mm to (396.9, 165.5)
- moved C14 1.26 mm to (386.1, 160.5)
- moved C26 1.26 mm to (388.8, 164.0)
- moved C28 1.26 mm to (393.3, 160.3)
- moved R1 1.26 mm to (383.4, 162.2)
- moved R2 1.26 mm to (381.5, 162.2)
- moved R3 1.26 mm to (390.6, 162.1)
- moved R4 1.26 mm to (388.7, 162.1)
- moved C13 1.26 mm to (381.5, 164.2)
- moved C15 1.26 mm to (386.1, 161.9)
- moved C27 1.26 mm to (393.3, 161.8)
- moved L2 1.26 mm to (385.6, 164.0)
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Routing:
- net /Camera/CSI_D1P: track 1.76 -> 14.3 mm
- net /Camera/CSI_D1N: track 2.74 -> 14.3 mm
- net /Camera/CSI_CKP: track 3.46 -> 14.5 mm
- net /Camera/CSI_D0P: track 2.85 -> 13.8 mm
- net /Camera/CSI_D0N: track 3.83 -> 13.9 mm
- net /Camera/CSI_CKN: track 4.66 -> 14.6 mm
- net /RF_915/SX_XTA: track 0.00 -> 4.11 mm
- net /RF_915/SX_XTB: track 0.00 -> 4.02 mm
- net /Camera/CSI_CON_CKN: track 0.00 -> 2.51 mm
- net /Camera/CSI_CON_CKP: track 0.00 -> 2.51 mm
- net /Camera/CSI_CON_D0N: track 0.00 -> 2.45 mm
- net /Camera/CSI_CON_D0P: track 0.00 -> 2.45 mm
- net /Camera/CSI_CON_D1P: track 0.00 -> 2.35 mm
- net /Camera/CSI_CON_D1N: track 0.00 -> 2.35 mm
- net GND: track 27.1 -> 26.1 mm, vias 181 -> 255
