File: hardware/drone/rf_915.kicad_sch (KiCad schematic)
At the start: 28 parts, among them U10 PE4259, U2 SX1262IMLTRT, U24 MM8030_2610RJ3, Y2 Crystal_GND24

Commit message: Continued footprint assignments
Parts:
- U24: footprint (none) -> SoftDroneLibrary:MM8030-2610RJ3
Changed lines of the file:
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@@
 			)
 		)
-		(property "Footprint" ""
+		(property "Footprint" "SoftDroneLibrary:MM8030-2610RJ3"
 			(at 238.76 86.36 0)
 			(hide yes)

Commit message: More footprints
Parts:
- C46, C47, C48, C50, C51, C52, C54, C56, C57, C61, C64, C65: footprint (none) -> Capacitor_SMD:C_0402_1005Metric
- C53: value 1.8 -> 1.8p; footprint (none) -> Capacitor_SMD:C_0402_1005Metric
- U10: footprint PE4259-63:SOT65P210X110-6N -> SoftDroneLibrary:PE4259
Changed lines of the file:
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@@
 			)
 		)
-		(property "Footprint" ""
+		(property "Footprint" "Capacitor_SMD:C_0402_1005Metric"
 			(at 223.8248 106.68 0)
 			(hide yes)
@@
 			)
 		)
-		(property "Footprint" ""
+		(property "Footprint" "Capacitor_SMD:C_0402_1005Metric"
 			(at 41.6052 46.99 0)
 			(hide yes)
@@
 			)
 		)
-		(property "Footprint" ""
+		(property "Footprint" "Capacitor_SMD:C_0402_1005Metric"
 			(at 125.4252 59.69 0)
 			(hide yes)
@@
 			)
 		)
-		(property "Footprint" ""
+		(property "Footprint" "Capacitor_SMD:C_0402_1005Metric"
 			(at 79.7052 46.99 0)
 			(hide yes)
@@
 			)
 		)
-		(property "Footprint" ""
+		(property "Footprint" "Capacitor_SMD:C_0402_1005Metric"
 			(at 177.8 71.4248 0)
 			(hide yes)
@@
 			)
 		)
-		(property "Footprint" ""
+		(property "Footprint" "Capacitor_SMD:C_0402_1005Metric"
 			(at 162.56 62.5348 0)
 			(hide yes)
@@
 			)
 		)
-		(property "Footprint" ""
+		(property "Footprint" "Capacitor_SMD:C_0402_1005Metric"
 			(at 135.5852 59.69 0)
 			(hide yes)
@@
 			)
 		)
-		(property "Footprint" ""
+		(property "Footprint" "Capacitor_SMD:C_0402_1005Metric"
 			(at 105.1052 67.31 0)
 			(hide yes)
@@
 			)
 		)
-		(property "Footprint" ""
+		(property "Footprint" "Capacitor_SMD:C_0402_1005Metric"
 			(at 167.3352 82.55 0)
 			(hide yes)
@@
 			)
 		)
-		(property "Footprint" ""
+		(property "Footprint" "Capacitor_SMD:C_0402_1005Metric"
 			(at 129.54 94.9452 0)
 			(hide yes)
@@
 			)
 		)
-		(property "Footprint" ""
+		(property "Footprint" "Capacitor_SMD:C_0402_1005Metric"
 			(at 51.7652 46.99 0)
 			(hide yes)
@@
 			)
 		)
-		(property "Footprint" ""
+		(property "Footprint" "Capacitor_SMD:C_0402_1005Metric"
 			(at 190.8048 74.93 0)
 			(hide yes)
@@
 			)
 		)
-		(property "Footprint" "PE4259-63:SOT65P210X110-6N"
+		(property "Footprint" "SoftDroneLibrary:PE4259"
 			(at 215.9 86.36 0)
 			(hide yes)
@@
 			)
 		)
-		(property "Value" "1.8"
+		(property "Value" "1.8p"
 			(at 128.27 110.4899 0)
 			(show_name no)
@@
 			)
 		)
-		(property "Footprint" ""
+		(property "Footprint" "Capacitor_SMD:C_0402_1005Metric"
 			(at 123.4948 105.41 0)
 			(hide yes)

Commit message: More footprints
Parts:
- C59, C60: footprint (none) -> Capacitor_SMD:C_0402_1005Metric
- L12: footprint (none) -> Inductor_SMD:L_0402_1005Metric
- R8: footprint (none) -> Resistor_SMD:R_0402_1005Metric
Changed lines of the file:
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@@
 			)
 		)
-		(property "Footprint" ""
+		(property "Footprint" "Resistor_SMD:R_0402_1005Metric"
 			(at 218.44 105.918 90)
 			(hide yes)
@@
 			)
 		)
-		(property "Footprint" ""
+		(property "Footprint" "Inductor_SMD:L_0402_1005Metric"
 			(at 260.35 86.36 0)
 			(hide yes)
@@
 			)
 		)
-		(property "Footprint" ""
+		(property "Footprint" "Capacitor_SMD:C_0402_1005Metric"
 			(at 250.4948 88.9 0)
 			(hide yes)
@@
 			)
 		)
-		(property "Footprint" ""
+		(property "Footprint" "Capacitor_SMD:C_0402_1005Metric"
 			(at 267.0048 88.9 0)
 			(hide yes)

Commit message: Completed footprint assignments
Parts:
- AE2: footprint (none) -> ANT-916-HETH:ANT916HETH
- L10, L6, L7, L8, L9: footprint (none) -> Inductor_SMD:L_0402_1005Metric
- L11: footprint (none) -> Inductor_SMD:L_0603_1608Metric
- Y2: footprint (none) -> Crystal:Crystal_SMD_3225-4Pin_3.2x2.5mm
Other:
- note added: "C362339"
- note added: "C486329"
Changed lines of the file:
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@@
 		)
 	)
+	(text "C486329"
+		(exclude_from_sim no)
+		(at 89.662 55.372 0)
+		(effects
+			(font
+				(size 1.27 1.27)
+			)
+		)
+	)
+	(text "C362339"
+		(exclude_from_sim no)
+		(at 20.574 43.688 0)
+		(effects
+			(font
+				(size 1.27 1.27)
+			)
+		)
+	)
 	(text "NRESET References VBAT"
 		(exclude_from_sim no)
@@
 			)
 		)
-		(property "Footprint" ""
+		(property "Footprint" "Crystal:Crystal_SMD_3225-4Pin_3.2x2.5mm"
 			(at 29.21 54.61 0)
 			(hide yes)
@@
 			)
 		)
-		(property "Footprint" ""
+		(property "Footprint" "ANT-916-HETH:ANT916HETH"
 			(at 274.32 78.74 0)
 			(hide yes)
@@
 			)
 		)
-		(property "Footprint" ""
+		(property "Footprint" "Inductor_SMD:L_0402_1005Metric"
 			(at 144.78 62.23 0)
 			(hide yes)
@@
 			)
 		)
-		(property "Footprint" ""
+		(property "Footprint" "Inductor_SMD:L_0402_1005Metric"
 			(at 124.46 99.06 0)
 			(hide yes)
@@
 			)
 		)
-		(property "Footprint" ""
+		(property "Footprint" "Inductor_SMD:L_0402_1005Metric"
 			(at 137.16 72.39 0)
 			(hide yes)
@@
 			)
 		)
-		(property "Footprint" ""
+		(property "Footprint" "Inductor_SMD:L_0402_1005Metric"
 			(at 185.42 72.39 0)
 			(hide yes)
@@
 			)
 		)
-		(property "Footprint" ""
+		(property "Footprint" "Inductor_SMD:L_0603_1608Metric"
 			(at 96.52 58.42 0)
 			(hide yes)
@@
 			)
 		)
-		(property "Footprint" ""
+		(property "Footprint" "Inductor_SMD:L_0402_1005Metric"
 			(at 158.75 72.39 0)
 			(hide yes)

Commit message: Labeled nets, added colours, and fixed stm32n6 schematic symbol issues
Connections:
- net SX_SW_CTRL: now reaches C61.2, R8.2, U10.4 (CTRL)
- net RFVRSUBG: now reaches C46.1, C47.1, L7.2, U2.24 (VR_PA)
- net RFISUBG_2: now reaches C53.2, L10.1, U2.21 (RFI_P)
- net RFISUBG_1: now reaches C54.2, L10.2, U2.22 (RFI_N)
- net RFOSUBG_1: now reaches L6.1, U2.23 (RFO)
- net SX_XTA: now reaches U2.3 (XTA), Y2.3
- net SX_XTB: now reaches U2.4 (XTB), Y2.1
- net RFCSUBG_ANT: now reaches AE2.1 (A), C60.2, L12.2
- net RFOSUBG_2: now reaches C48.1, L6.2, L7.1, L8.1
- net RFCSUBG_2: now reaches C59.2, L12.1, U24.2 (OUT)
- net RFOSUBG_3: now reaches C48.2, C50.1, C51.1, L8.2
- net RFOSUBG_4: now reaches C51.2, L9.1
- net RFOSUBG_5: now reaches C52.2, L9.2, U10.1 (RF1)
- net RFISUBG_3: now reaches C54.1, U10.3 (RF2)
- net RFCSUBG_1: now reaches U10.5 (RFC), U24.1 (IN)
Other:
- moved on the sheet: C52, L9
Changed lines of the file:
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@@
 	)
 	(junction
-		(at 191.77 72.39)
+		(at 194.31 72.39)
 		(diameter 0)
 		(color 0 0 0 0)
@@
 	(wire
 		(pts
-			(xy 191.77 74.93) (xy 191.77 72.39)
+			(xy 194.31 74.93) (xy 194.31 72.39)
 		)
 		(stroke
@@
 	(wire
 		(pts
-			(xy 191.77 82.55) (xy 191.77 83.82)
+			(xy 194.31 82.55) (xy 194.31 83.82)
 		)
 		(stroke
@@
 	(wire
 		(pts
-			(xy 224.79 86.36) (xy 229.87 86.36)
-		)
-		(stroke
-			(width 0)
-			(type default)
-		)
-	)
-	(wire
-		(pts
 			(xy 104.14 59.69) (xy 104.14 58.42)
 		)
@@
 	(wire
 		(pts
-			(xy 125.73 81.28) (xy 125.73 72.39)
+			(xy 224.79 86.36) (xy 229.87 86.36)
 		)
 		(stroke
@@
 	(wire
 		(pts
-			(xy 189.23 72.39) (xy 191.77 72.39)
+			(xy 125.73 81.28) (xy 125.73 72.39)
 		)
 		(stroke
@@
 	(wire
 		(pts
-			(xy 177.8 72.39) (xy 181.61 72.39)
+			(xy 177.8 72.39) (xy 184.15 72.39)
 		)
 		(stroke
@@
 		)
 	)
+	(label "RFISUBG_3"
+		(at 142.24 93.98 0)
+		(effects
+			(font
+				(size 1.27 1.27)
+			)
+			(justify left bottom)
+		)
+	)
+	(label "RFCSUBG_ANT"
+		(at 265.43 86.36 0)
+		(effects
+			(font
+				(size 0.635 0.635)
+			)
+			(justify left bottom)
+		)
+	)
+	(label "RFCSUBG_2"
+		(at 248.92 86.36 0)
+		(effects
+			(font
+				(size 0.635 0.635)
+			)
+			(justify left bottom)
+		)
+	)
+	(label "SX_SW_CTRL"
+		(at 228.6 102.87 90)
+		(effects
+			(font
+				(size 1.27 1.27)
+			)
+			(justify left bottom)
+		)
+	)
+	(label "RFOSUBG_2"
+		(at 142.24 72.39 0)
+		(effects
+			(font
+				(size 0.635 0.635)
+			)
+			(justify left bottom)
+		)
+	)
+	(label "RFCSUBG_1"
+		(at 224.79 86.36 0)
+		(effects
+			(font
+				(size 0.635 0.635)
+			)
+			(justify left bottom)
+		)
+	)
+	(label "RFVRSUBG"
+		(at 87.63 73.66 0)
+		(effects
+			(font
+				(size 1.27 1.27)
+			)
+			(justify left bottom)
+		)
+	)
+	(label "RFOSUBG_5"
+		(at 195.58 72.39 0)
+		(effects
+			(font
+				(size 0.635 0.635)
+			)
+			(justify left bottom)
+		)
+	)
 	(label "SX_DIO2"
 		(at 35.56 81.28 0)
@@
 		)
 	)
+	(label "RFOSUBG_3"
+		(at 163.83 72.39 0)
+		(effects
+			(font
+				(size 0.635 0.635)
+			)
+			(justify left bottom)
+		)
+	)
 	(label "SX_DIO2"
 		(at 203.2 104.14 0)
@@
 		)
 	)
+	(label "RFOSUBG_4"
+		(at 177.8 72.39 0)
+		(effects
+			(font
+				(size 0.635 0.635)
+			)
+			(justify left bottom)
+		)
+	)
+	(label "RFOSUBG_1"
+		(at 87.63 81.28 0)
+		(effects
+			(font
+				(size 1.27 1.27)
+			)
+			(justify left bottom)
+		)
+	)
+	(label "RFISUBG_2"
+		(at 87.63 86.36 0)
+		(effects
+			(font
+				(size 1.27 1.27)
+			)
+			(justify left bottom)
+		)
+	)
+	(label "SX_XTB"
+		(at 38.1 68.58 0)
+		(effects
+			(font
+				(size 1.27 1.27)
+			)
+			(justify left bottom)
+		)
+	)
+	(label "SX_XTA"
+		(at 38.1 66.04 0)
+		(effects
+			(font
+				(size 1.27 1.27)
+			)
+			(justify left bottom)
+		)
+	)
+	(label "RFISUBG_1"
+		(at 87.63 83.82 0)
+		(effects
+			(font
+				(size 1.27 1.27)
+			)
+			(justify left bottom)
+		)
+	)
 	(global_label "SX_NRST"
 		(shape input)
@@
 	(symbol
 		(lib_id "Device:L")
-		(at 185.42 72.39 90)
+		(at 187.96 72.39 90)
 		(unit 1)
 		(body_style 1)
@@
 		(fields_autoplaced yes)
 		(property "Reference" "L9"
-			(at 185.42 67.31 90)
+			(at 187.96 67.31 90)
 			(show_name no)
 			(do_not_autoplace no)
@@
 		)
 		(property "Value" "4.7n"
-			(at 185.42 69.85 90)
+			(at 187.96 69.85 90)
 			(show_name no)
 			(do_not_autoplace no)
@@
 		)
 		(property "Footprint" "Inductor_SMD:L_0402_1005Metric"
-			(at 185.42 72.39 0)
+			(at 187.96 72.39 0)
 			(hide yes)
 			(show_name no)
@@
 		)
 		(property "Datasheet" ""
-			(at 185.42 72.39 0)
+			(at 187.96 72.39 0)
 			(hide yes)
 			(show_name no)
@@
 		)
 		(property "Description" "Inductor"
-			(at 185.42 72.39 0)
+			(at 187.96 72.39 0)
 			(hide yes)
 			(show_name no)
@@
 	(symbol
 		(lib_id "Device:C")
-		(at 191.77 78.74 180)
+		(at 194.31 78.74 180)
 		(unit 1)
 		(body_style 1)
@@
 		(fields_autoplaced yes)
 		(property "Reference" "C52"
-			(at 195.58 77.4699 0)
+			(at 198.12 77.4699 0)
 			(show_name no)
 			(do_not_autoplace no)
@@
 		)
 		(property "Value" "1.8p"
-			(at 195.58 80.0099 0)
+			(at 198.12 80.0099 0)
 			(show_name no)
 			(do_not_autoplace no)
@@
 		)
 		(property "Footprint" "Capacitor_SMD:C_0402_1005Metric"
-			(at 190.8048 74.93 0)
+			(at 193.3448 74.93 0)
 			(hide yes)
 			(show_name no)
@@
 		)
 		(property "Datasheet" ""
-			(at 191.77 78.74 0)
+			(at 194.31 78.74 0)
 			(hide yes)
 			(show_name no)
@@
 		)
 		(property "Description" "Unpolarized capacitor"
-			(at 191.77 78.74 0)
+			(at 194.31 78.74 0)
 			(hide yes)
 			(show_name no)
@@
 	(symbol
 		(lib_id "power:GND")
-		(at 191.77 83.82 0)
+		(at 194.31 83.82 0)
 		(unit 1)
 		(body_style 1)
@@
 		(in_pos_files yes)
 		(dnp no)
-		(fields_autoplaced yes)
 		(property "Reference" "#PWR073"
-			(at 191.77 90.17 0)
+			(at 194.31 90.17 0)
 			(hide yes)
 			(show_name no)
@@
 		)
 		(property "Value" "GND"
-			(at 191.77 88.9 0)
+			(at 189.992 86.614 0)
 			(show_name no)
 			(do_not_autoplace no)
@@
 		)
 		(property "Footprint" ""
-			(at 191.77 83.82 0)
+			(at 194.31 83.82 0)
 			(hide yes)
 			(show_name no)
@@
 		)
 		(property "Datasheet" ""
-			(at 191.77 83.82 0)
+			(at 194.31 83.82 0)
 			(hide yes)
 			(show_name no)
@@
 		)
 		(property "Description" "Power symbol creates a global label with name \"GND\" , ground"
-			(at 191.77 83.82 0)
+			(at 194.31 83.82 0)
 			(hide yes)
 			(show_name no)

Commit message: Started layout and tested RF routing paths
Parts:
- C59, C60: footprint Capacitor_SMD:C_0402_1005Metric -> Capacitor_SMD:C_0603_1608Metric
- L12: footprint Inductor_SMD:L_0402_1005Metric -> Inductor_SMD:L_0603_1608Metric
Changed lines of the file:
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@@
 			)
 		)
-		(property "Footprint" "Inductor_SMD:L_0402_1005Metric"
+		(property "Footprint" "Inductor_SMD:L_0603_1608Metric"
 			(at 260.35 86.36 0)
 			(hide yes)
@@
 			)
 		)
-		(property "Footprint" "Capacitor_SMD:C_0402_1005Metric"
+		(property "Footprint" "Capacitor_SMD:C_0603_1608Metric"
 			(at 250.4948 88.9 0)
 			(hide yes)
@@
 			)
 		)
-		(property "Footprint" "Capacitor_SMD:C_0402_1005Metric"
+		(property "Footprint" "Capacitor_SMD:C_0603_1608Metric"
 			(at 267.0048 88.9 0)
 			(hide yes)

Commit message: Routed OSPI
Connections:
- net SX_DCC_SW: now reaches L11.1, U2.9 (DCC_SW)
Changed lines of the file:
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@@
+		)
+	)
+	(label "SX_DCC_SW"
+		(at 81.28 68.58 0)
+		(effects
+			(font
+				(size 0.762 0.762)
+			)
+			(justify left bottom)
 		)
 	)

Commit message: SX1262 layout and decoupling
Parts:
- C57, C64, C65: footprint Capacitor_SMD:C_0402_1005Metric -> Capacitor_SMD:C_0201_0603Metric
Connections:
- net SX_DCC_SW renamed SX_SMPS_SW
Changed lines of the file:
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@@
 		)
 	)
-	(label "SX_DCC_SW"
+	(label "SX_SMPS_SW"
 		(at 81.28 68.58 0)
 		(effects
@@
 			)
 		)
-		(property "Footprint" "Capacitor_SMD:C_0402_1005Metric"
+		(property "Footprint" "Capacitor_SMD:C_0201_0603Metric"
 			(at 41.6052 46.99 0)
 			(hide yes)
@@
 			)
 		)
-		(property "Footprint" "Capacitor_SMD:C_0402_1005Metric"
+		(property "Footprint" "Capacitor_SMD:C_0201_0603Metric"
 			(at 79.7052 46.99 0)
 			(hide yes)
@@
 			)
 		)
-		(property "Footprint" "Capacitor_SMD:C_0402_1005Metric"
+		(property "Footprint" "Capacitor_SMD:C_0201_0603Metric"
 			(at 51.7652 46.99 0)
 			(hide yes)
