File: hardware/drone/rf_915.kicad_sch (KiCad schematic)
At the start: 28 parts, among them U10 PE4259, U2 SX1262IMLTRT, U24 MM8030_2610RJ3, Y2 Crystal_GND24

Commit message: Started power routing
Parts:
- added C126, C87: C, Capacitor_SMD:C_0402_1005Metric, symbol Device:C
Connections:
- net GND: now also C126.2, C87.2
- net RFISUBG_3: now also C126.1
- net RFOSUBG_2: now also C87.1

Commit message: Small cleanup and more power routing
Changed lines of the file:
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@@
 	(generator_version "10.0")
 	(paper "A4")
+	(rectangle
+		(start 14.605 17.145)
+		(end 281.94 127)
+		(stroke
+			(width 0)
+			(type default)
+		)
+		(fill
+			(type none)
+		)
+	)
 	(text "SX1262 915MHz Radio"
 		(exclude_from_sim no)

Commit message: more power layout
Connections:
- net SX_VREG: now reaches C56.1, L11.2, U2.7 (VREG)
Changed lines of the file:
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@@
+		)
+	)
+	(label "SX_VREG"
+		(at 85.09 50.8 0)
+		(effects
+			(font
+				(size 0.762 0.762)
+			)
+			(justify left bottom)
 		)
 	)

Commit message: Schematic cleanup and changed pi network footprints
Parts:
- C59, C60: now not fitted
- L12: value L -> 0
Changed lines of the file:
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@@
 			)
 		)
-		(property "Value" "L"
+		(property "Value" "0"
 			(at 260.35 83.82 90)
 			(show_name no)
@@
 		(on_board yes)
 		(in_pos_files yes)
-		(dnp no)
+		(dnp yes)
 		(fields_autoplaced yes)
 		(property "Reference" "C59"
@@
 		(on_board yes)
 		(in_pos_files yes)
-		(dnp no)
+		(dnp yes)
 		(fields_autoplaced yes)
 		(property "Reference" "C60"
