File: hardware/drone/_restore_backup_2026-09-17T12-52-13-706/audio.kicad_sch (KiCad schematic)
At the start: 21 parts, among them J6 Conn_01x02_Socket, U11 TAC5111IRGER, U28 LM4670ITL/NOPB

Commit message: Codec layout
Parts:
- C73, C74: footprint Capacitor_SMD:C_0402_1005Metric -> Capacitor_SMD:C_0603_1608Metric
- C76, C77: footprint Capacitor_SMD:C_0201_0603Metric -> Capacitor_SMD:C_0603_1608Metric
- R10, R9: footprint Resistor_SMD:R_0201_0603Metric -> Resistor_SMD:R_0603_1608Metric
Connections:
- net CODEC_SPK1: now also J6.1 (Pin_1); no longer J6.2 (Pin_2)
- net CODEC_SPK2: now also J6.2 (Pin_2); no longer J6.1 (Pin_1)
- net CODEC_DREG: no longer names the net of C69.1, C70.1, U11.1 (DREG)
- net CODEC_MEM_IN1N renamed CODEC_MEM_IN1M
- net CODEC_MEM_IN1N_1 renamed CODEC_MEM_IN1M_1
- net CODEC_OUT1N renamed CODEC_OUT1M
- net CODEC_OUT1N_1 renamed CODEC_OUT1M_1
- net CODEC_OUT1N_2 renamed CODEC_OUT1M_2
- net CODEC_VREF: no longer names the net of C68.1, U11.24 (VREF)
Changed lines of the file:
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@@
-		)
-	)
-	(label "CODEC_DREG"
-		(at 128.27 33.02 0)
-		(effects
-			(font
-				(size 0.635 0.635)
-			)
-			(justify left bottom)
 		)
 	)
@@
 		)
 	)
-	(label "CODEC_OUT1N"
+	(label "CODEC_OUT1M"
 		(at 148.59 82.55 0)
 		(effects
@@
 		)
 	)
-	(label "CODEC_OUT1N_1"
+	(label "CODEC_OUT1M_1"
 		(at 163.83 85.09 0)
 		(effects
@@
 		)
 	)
-	(label "CODEC_VREF"
-		(at 111.76 33.02 0)
-		(effects
-			(font
-				(size 0.635 0.635)
-			)
-			(justify left bottom)
-		)
-	)
-	(label "CODEC_OUT1N_2"
+	(label "CODEC_OUT1M_2"
 		(at 176.53 85.09 0)
 		(effects
@@
 		)
 	)
-	(label "CODEC_MEM_IN1N"
+	(label "CODEC_MEM_IN1M"
 		(at 86.36 82.55 0)
 		(effects
@@
 		)
 	)
-	(label "CODEC_MEM_IN1N_1"
+	(label "CODEC_MEM_IN1M_1"
 		(at 59.69 82.55 0)
 		(effects
@@
 			)
 		)
-		(property "Footprint" "Capacitor_SMD:C_0201_0603Metric"
+		(property "Footprint" "Capacitor_SMD:C_0603_1608Metric"
 			(at 163.83 76.5048 0)
 			(hide yes)
@@
 			)
 		)
-		(property "Footprint" "Resistor_SMD:R_0201_0603Metric"
+		(property "Footprint" "Resistor_SMD:R_0603_1608Metric"
 			(at 172.72 79.248 90)
 			(hide yes)
@@
 			)
 		)
-		(property "Footprint" "Capacitor_SMD:C_0402_1005Metric"
+		(property "Footprint" "Capacitor_SMD:C_0603_1608Metric"
 			(at 81.28 76.5048 0)
 			(hide yes)
@@
 			)
 		)
-		(property "Footprint" "Capacitor_SMD:C_0201_0603Metric"
+		(property "Footprint" "Capacitor_SMD:C_0603_1608Metric"
 			(at 156.21 84.1248 0)
 			(hide yes)
@@
 	(symbol
 		(lib_id "Connector:Conn_01x02_Socket")
-		(at 232.41 80.01 0)
+		(at 232.41 82.55 0)
+		(mirror x)
 		(unit 1)
 		(body_style 1)
@@
 		(dnp no)
 		(property "Reference" "J6"
-			(at 233.68 80.0099 0)
+			(at 233.68 82.5501 0)
 			(show_name no)
 			(do_not_autoplace no)
@@
 		)
 		(property "Value" "Conn_01x02_Socket"
-			(at 233.68 82.5499 0)
+			(at 233.68 80.0101 0)
 			(show_name no)
 			(do_not_autoplace no)
@@
 		)
 		(property "Footprint" "Connector_JST:JST_SH_BM02B-SRSS-TB_1x02-1MP_P1.00mm_Vertical"
-			(at 232.41 80.01 0)
-			(hide yes)
-			(show_name no)
-			(do_not_autoplace no)
-			(effects
-				(font
-					(size 1.27 1.27)
-				)
-			)
-		)
-		(property "Datasheet" ""
-			(at 232.41 80.01 0)
+			(at 232.41 82.55 0)
+			(hide yes)
+			(show_name no)
+			(do_not_autoplace no)
+			(effects
+				(font
+					(size 1.27 1.27)
+				)
+			)
+		)
+		(property "Datasheet" ""
+			(at 232.41 82.55 0)
 			(hide yes)
 			(show_name no)
@@
 		)
 		(property "Description" "Generic connector, single row, 01x02, script generated"
-			(at 232.41 80.01 0)
+			(at 232.41 82.55 0)
 			(hide yes)
 			(show_name no)
@@
 			)
 		)
-		(property "Footprint" "Resistor_SMD:R_0201_0603Metric"
+		(property "Footprint" "Resistor_SMD:R_0603_1608Metric"
 			(at 172.72 83.312 90)
 			(hide yes)
@@
 			)
 		)
-		(property "Footprint" "Capacitor_SMD:C_0402_1005Metric"
+		(property "Footprint" "Capacitor_SMD:C_0603_1608Metric"
 			(at 81.28 86.0552 0)
 			(hide yes)
