File: hardware/drone/_restore_backup_2026-09-17T12-52-13-706/drone.kicad_pcb (KiCad board)
At the start: 6 copper layers, 80 x 50 mm, 244 parts, among them J1 54548-2272, J2 BM08B-SRSS-TB_LF__SN_, J3 USB_C_Receptacle_USB2.0_16P, J4 Conn_ARM_SWD_TagConnect_TC2030, J5 Conn_01x06_Pin, J6 Conn_01x02_Socket, SW1 SW_MEC_5E, U1 STM32N645I0, U10 PE4259, U11 TAC5111IRGER, U12 LP5907, U13 SQA411CEJW-T1_GE3, U14 ICM-42688-P, U15 SAM_M10Q, U16 LMR51635YFDDCR, U17 TXU0204, U18 TPS2121, U19 BMP581, U2 SX1262IMLTRT, U20 TVS0500DRV, U21 TCA9406DC, U22 LIS2MDL, U23 MM8030_2610RJ3, U24 MM8030_2610RJ3, U25 ECMF2-40A100N6, U26 ECMF2-40A100N6, U27 ECMF2-40A100N6, U28 LM4670ITL/NOPB, U3 TPS628303, U4 TPS7A2118PQWDSGRQ1, U5 TPS628303, U6 MX25UW25645GXDI00, U7 CC3350, U8 DPX167125DT-8197B1, U9 DEA162450BT-1295A1, Y1 Crystal_GND24, Y2 Crystal_GND24, Y3 Crystal_GND24, Y4 Crystal

Commit message: Codec layout
Parts:
- C73, C74: footprint Capacitor_SMD:C_0402_1005Metric -> Capacitor_SMD:C_0603_1608Metric; moved to F.Cu
- C76, C77: footprint Capacitor_SMD:C_0201_0603Metric -> Capacitor_SMD:C_0603_1608Metric
- MK2, U15: moved to F.Cu
- R10, R9: footprint Resistor_SMD:R_0201_0603Metric -> Resistor_SMD:R_0603_1608Metric
- U11: moved to B.Cu
- moved U14 265.0 mm to (141.6, 191.7)
- moved U22 264.7 mm to (123.9, 180.9)
- moved C80 249.7 mm to (123.8, 255.6)
- moved C81 249.2 mm to (123.8, 257.6)
- moved U19 244.9 mm to (149.9, 236.7)
- moved MK2 244.8 mm to (107.9, 191.1), turned to 0 degrees
- moved U28 212.1 mm to (143.8, 175.8), turned to 0 degrees
- moved U12 189.8 mm to (166.4, 129.2), turned to 0 degrees
- moved R10 182.5 mm to (203.4, 256.5), turned to 0 degrees
- moved R9 181.5 mm to (203.4, 254.0), turned to 0 degrees
- moved C77 178.5 mm to (203.4, 246.4)
- moved C76 177.6 mm to (203.4, 243.9), turned to 0 degrees
- moved C74 170.8 mm to (203.4, 241.4)
- moved C73 170.0 mm to (203.4, 238.9)
- moved J6 167.0 mm to (187.6, 190.7), turned to 0 degrees
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Connections:
- net /Audio/CODEC_DREG renamed Net-(U11-DREG)
- net /Audio/CODEC_MEM_IN1N renamed /Audio/CODEC_MEM_IN1M
- net /Audio/CODEC_MEM_IN1N_1 renamed /Audio/CODEC_MEM_IN1M_1
- net /Audio/CODEC_OUT1N renamed /Audio/CODEC_OUT1M
- net /Audio/CODEC_OUT1N_1 renamed /Audio/CODEC_OUT1M_1
- net /Audio/CODEC_OUT1N_2 renamed /Audio/CODEC_OUT1M_2
- net /Audio/CODEC_VREF renamed Net-(U11-VREF)
- J6 pad 1: /Audio/CODEC_SPK2 -> /Audio/CODEC_SPK1
- J6 pad 2: /Audio/CODEC_SPK1 -> /Audio/CODEC_SPK2
Routing:
- net CC_SDMMC1_D2: track 47.8 -> 36.0 mm
- net CC_SDMMC1_D3: track 41.8 -> 35.3 mm
- net CC_SDMMC1_CLK: track 43.0 -> 36.7 mm
- net CC_SDMMC1_CMD: track 46.9 -> 40.8 mm
- net CC_SDMMC1_D0: track 49.1 -> 43.0 mm
- net CC_SDMMC1_D1: track 44.2 -> 39.0 mm
- net IMU_CS: track 3.32 -> 0.00 mm, vias 1 -> 0
- net IMU_SPI4_MOSI: track 2.17 -> 0.00 mm, vias 1 -> 0
- net IMU_SPI4_MISO: track 2.16 -> 0.00 mm, vias 1 -> 0
- net /Audio/CODEC_MEM_IN1P_1: track 2.16 -> 0.00 mm
- net /Audio/CODEC_MEM_IN1M_1: track 2.16 -> 0.00 mm
- net IMU_SPI4_SCK: track 1.48 -> 0.00 mm, vias 1 -> 0
- net VSYS_5V: track 0.92 -> 0.00 mm, vias 1 -> 0
- net GND: vias 306 -> 255
